Commit message: everything working in robot_description

File: robot_description/model/robots/robot_3d.urdf.xacro (robot description, xacro)
@@ -31,9 +31,4 @@
       x_reflect="-1"
       y_reflect="-1"/>
-    <xacro:rgbd_camera
-      prefix="$(arg prefix)"
-      camera_name="cam_1"
-      xyz_offset="0.105 0 0.03"
-      rpy_offset="0 0 0"/>
     <xacro:lidar_sensor
       prefix="$(arg prefix)"
@@ -42,6 +37,4 @@
       xyz_offset="0 0 0.0825"
       rpy_offset="0 0 3.14"
-      mesh_xyz_offset="0 0 0"
-      mesh_rpy_offset="${-M_PI/2} 0 0"
       topic_name="scan"/>
     <xacro:imu_sensor

File: robot_description/model/sensors/lidar.urdf.xacro (robot description, xacro)
@@ -6,10 +6,6 @@
     parent:='base_link'
     frame_id:='laser_frame'
-    mesh_file:='file://$(find mec_mobile_description)/meshes/rplidar/rplidar_s2.stl'
     xyz_offset:='0 0 0.0825'
     rpy_offset:='0 0 0'
-    mesh_xyz_offset:='0 0 0'
-    mesh_rpy_offset:='${-M_PI/2} 0 0'
-    mesh_scale:='0.001 0.001 0.001'
     collision_xyz_offset:='0 0 0'
     collision_rpy_offset:='0 0 0'
@@ -40,7 +36,7 @@
     <link name="${prefix}${frame_id}">
       <visual>
-        <origin xyz="${mesh_xyz_offset}" rpy="${mesh_rpy_offset}"/>
+        <origin xyz="0 0 ${lidar_height/2}" rpy="0 0 0"/>
         <geometry>
-          <mesh filename="${mesh_file}" scale="${mesh_scale}"/>
+          <cylinder radius="${radius}" length="${lidar_height}"/>
         </geometry>
         <material name="${material_name}">
@@ -50,7 +46,7 @@
       <xacro:if value="${enable_collision}">
         <collision>
-          <origin xyz="${collision_xyz_offset}" rpy="${collision_rpy_offset}"/>
+          <origin xyz="0 0 ${lidar_height/2}" rpy="0 0 0"/>
           <geometry>
-            <cylinder radius="${lidar_width/2}" length="${lidar_height}"/>
+            <cylinder radius="${radius}" length="${lidar_height}"/>
           </geometry>
         </collision>

Commit message: without prefix working

File: robot_description/model/robots/robot_3d.urdf.xacro (robot description, xacro)
@@ -10,4 +10,5 @@
     <xacro:include filename="$(find robot_description)/model/control/robot.gazebo"/>
     <xacro:robot_3d_base prefix="$(arg prefix)"/>
+    <xacro:robot_gazebo prefix="$(arg prefix)" />
     <xacro:mecanum_wheel
       prefix="$(arg prefix)"
@@ -100,5 +101,4 @@
     <mu1>0.000002</mu1>
     <mu2>0.000002</mu2>
-    <!-- <material>Gazebo/Red</material> -->
   </gazebo>
 </robot>

Commit message: added controlling every robot

File: robot_description/model/robots/robot_3d.urdf.xacro (robot description, xacro)
@@ -10,5 +10,6 @@
     <xacro:include filename="$(find robot_description)/model/control/robot.gazebo"/>
     <xacro:robot_3d_base prefix="$(arg prefix)"/>
-    <xacro:robot_gazebo prefix="$(arg prefix)" />
+<xacro:property name="prefix" value="$(arg prefix)" />
+    <xacro:robot_gazebo prefix="${prefix}" />
     <xacro:mecanum_wheel
       prefix="$(arg prefix)"
@@ -46,5 +47,5 @@
       update_rate="15.0"
       topic_name="imu/data"/>
-  <gazebo reference='front_left_wheel_link'>
+  <gazebo reference='${prefix}front_left_wheel_link'>
     <collision>
       <surface>
@@ -53,5 +54,5 @@
             <mu>1.5</mu>
             <mu2>0.0</mu2>
-            <fdir1 gz:expressed_in="base_footprint">1 -1 0</fdir1>
+            <fdir1 gz:expressed_in="${prefix}base_footprint">1 -1 0</fdir1>
           </ode>
         </friction>
@@ -59,5 +60,5 @@
     </collision>
   </gazebo>
-  <gazebo reference='back_left_wheel_link'>
+  <gazebo reference='${prefix}back_left_wheel_link'>
     <collision>
       <surface>
@@ -66,5 +67,5 @@
             <mu>1.5</mu>
             <mu2>0.0</mu2>
-            <fdir1 gz:expressed_in="base_footprint">1 1 0</fdir1>
+            <fdir1 gz:expressed_in="${prefix}base_footprint">1 1 0</fdir1>
           </ode>
         </friction>
@@ -72,5 +73,5 @@
     </collision>
   </gazebo>
-  <gazebo reference='front_right_wheel_link'>
+  <gazebo reference='${prefix}front_right_wheel_link'>
     <collision>
       <surface>
@@ -79,5 +80,5 @@
             <mu>1.5</mu>
             <mu2>0.0</mu2>
-            <fdir1 gz:expressed_in="base_footprint">1 1 0</fdir1>
+            <fdir1 gz:expressed_in="${prefix}base_footprint">1 1 0</fdir1>
           </ode>
         </friction>
@@ -85,5 +86,5 @@
     </collision>
   </gazebo>
-  <gazebo reference='back_right_wheel_link'>
+  <gazebo reference='${prefix}back_right_wheel_link'>
     <collision>
       <surface>
@@ -92,5 +93,5 @@
             <mu>1.5</mu>
             <mu2>0.0</mu2>
-            <fdir1 gz:expressed_in="base_footprint">1 -1 0</fdir1>
+            <fdir1 gz:expressed_in="${prefix}base_footprint">1 -1 0</fdir1>
           </ode>
         </friction>
@@ -98,5 +99,5 @@
     </collision>
   </gazebo>
-  <gazebo reference="base_link">
+  <gazebo reference="${prefix}base_link">
     <mu1>0.000002</mu1>
     <mu2>0.000002</mu2>

Commit message: added scan and imu to swarm

File: robot_description/model/robots/robot_3d.urdf.xacro (robot description, xacro)
@@ -4,4 +4,5 @@
     <xacro:arg name="robot_name" default="robot_3d"/>
     <xacro:arg name="prefix" default=""/>
+    <xacro:property name="prefix" value="$(arg prefix)" />
     <xacro:include filename="$(find robot_description)/model/mech/robot_3d_base.urdf.xacro"/>
     <xacro:include filename="$(find robot_description)/model/mech/mecanum_wheel.urdf.xacro"/>
@@ -10,5 +11,4 @@
     <xacro:include filename="$(find robot_description)/model/control/robot.gazebo"/>
     <xacro:robot_3d_base prefix="$(arg prefix)"/>
-<xacro:property name="prefix" value="$(arg prefix)" />
     <xacro:robot_gazebo prefix="${prefix}" />
     <xacro:mecanum_wheel

File: robot_description/model/sensors/imu.urdf.xacro (robot description, xacro)
@@ -60,5 +60,5 @@
             </material>
             <sensor name="${prefix}imu_sensor" type="imu">
-                <topic>${topic_name}</topic>
+                <topic>${prefix}${topic_name}</topic>
                 <update_rate>${update_rate}</update_rate>
                 <always_on>${always_on}</always_on>

File: robot_description/model/sensors/lidar.urdf.xacro (robot description, xacro)
@@ -76,5 +76,5 @@
       </material>
       <sensor name="${prefix}lidar_sensor" type="gpu_lidar">
-        <topic>${topic_name}</topic>
+        <topic>${prefix}${topic_name}</topic>
         <update_rate>${update_rate}</update_rate>
         <always_on>${always_on}</always_on>
